File: chessboard_controller/chessboard_controller.kicad_pcb (KiCad board)
At the start: 2 copper layers, 13 parts, among them J1 Conn_01x04, J2 Conn_01x06, J3 Conn_01x08, J4 Conn_01x08, J5 Conn_01x10, U1 HV4067, U2 HV4067, U3 HV4067, U4 HV4067

Commit message: First version of layout
Parts:
- removed H3, H4: MountingHole, MountingHole:MountingHole_3.2mm_M3
- added J6: Conn_02x17_Counter_Clockwise, Connector_IDC:IDC-Header_2x17_P2.54mm_Horizontal, F.Cu at (101.9, 102.4)
- added J7: Conn_02x17_Counter_Clockwise, Connector_IDC:IDC-Header_2x17_P2.54mm_Horizontal, F.Cu at (199.1, 61.7)
- H1, H2: footprint MountingHole:MountingHole_3.2mm_M3 -> MountingHole:MountingHole_3.2mm_M3_ISO7380
- moved H2 153.6 mm to (118.4, 106.2)
- moved U4 116.0 mm to (196.8, 91.9)
- moved U2 112.2 mm to (152.4, 71.9), turned to -90 degrees
- moved J5 92.9 mm to (123.2, 58.0)
- moved J2 92.9 mm to (155.2, 106.2)
- moved J3 92.9 mm to (132.3, 106.2)
- moved J4 92.9 mm to (150.1, 58.0)
- moved H1 92.8 mm to (119.6, 57.9)
- moved U1 74.0 mm to (152.4, 91.9), turned to -90 degrees
- moved J1 64.8 mm to (106.7, 58.0), turned to 90 degrees
- moved U3 16.3 mm to (196.8, 71.9), turned to -90 degrees
Connections:
- net /D0_Rx renamed /RX/D0
- net /D1_Tx renamed /TX/D1
- net /D2 renamed /S0
- net /D3 renamed /S1
- net /D4 renamed /S2
- net /D5 renamed /S3
- net /RES renamed /~{RESET}
- net /VIN renamed VCC
- J1 pad 3: /SDA -> /SDA/A4
- J1 pad 4: /SCL -> /SCL/A5
- J2 pad 5: /A4 -> /SDA
- J2 pad 6: /A5 -> /SCL
- J3 pad 2: +5V -> /IOREF
- J5 pad 1: /SCL -> /SCL/A5
- J5 pad 2: /SDA -> /SDA/A4
- U1 pad 10: unconnected-(U1-C1-Pad10) -> /c102
- U1 pad 11: unconnected-(U1-C2-Pad11) -> /c103
- U1 pad 12: unconnected-(U1-C3-Pad12) -> /c104
- U1 pad 13: unconnected-(U1-C4-Pad13) -> /c105
- U1 pad 14: unconnected-(U1-C5-Pad14) -> /c106
- U1 pad 15: unconnected-(U1-C6-Pad15) -> /c107
- U1 pad 16: unconnected-(U1-C7-Pad16) -> /c108
- U1 pad 17: unconnected-(U1-C8-Pad17) -> /c109
- U1 pad 18: unconnected-(U1-C9-Pad18) -> /c110
- U1 pad 19: unconnected-(U1-C10-Pad19) -> /c111
- U1 pad 20: unconnected-(U1-C11-Pad20) -> /c112
- U1 pad 21: unconnected-(U1-C12-Pad21) -> /c113
- U1 pad 22: unconnected-(U1-C13-Pad22) -> /c114
- U1 pad 23: unconnected-(U1-C14-Pad23) -> /c115
- U1 pad 24: unconnected-(U1-C15-Pad24) -> /c116
- U1 pad 9: unconnected-(U1-C0-Pad9) -> /c101
- U2 pad 10: unconnected-(U2-C1-Pad10) -> /c202
- U2 pad 11: unconnected-(U2-C2-Pad11) -> /c203
- U2 pad 12: unconnected-(U2-C3-Pad12) -> /c204
- U2 pad 13: unconnected-(U2-C4-Pad13) -> /c205
- U2 pad 14: unconnected-(U2-C5-Pad14) -> /c206
- U2 pad 15: unconnected-(U2-C6-Pad15) -> /c207
- U2 pad 16: unconnected-(U2-C7-Pad16) -> /c208
- U2 pad 17: unconnected-(U2-C8-Pad17) -> /c209
- U2 pad 18: unconnected-(U2-C9-Pad18) -> /c210
- U2 pad 19: unconnected-(U2-C10-Pad19) -> /c211
- U2 pad 20: unconnected-(U2-C11-Pad20) -> /c212
- U2 pad 21: unconnected-(U2-C12-Pad21) -> /c213
- U2 pad 22: unconnected-(U2-C13-Pad22) -> /c214
- U2 pad 23: unconnected-(U2-C14-Pad23) -> /c215
- U2 pad 24: unconnected-(U2-C15-Pad24) -> /c216
- U2 pad 9: unconnected-(U2-C0-Pad9) -> /c201
- U3 pad 10: unconnected-(U3-C1-Pad10) -> /c302
- U3 pad 11: unconnected-(U3-C2-Pad11) -> /c303
- U3 pad 12: unconnected-(U3-C3-Pad12) -> /c304
- U3 pad 13: unconnected-(U3-C4-Pad13) -> /c305
- U3 pad 14: unconnected-(U3-C5-Pad14) -> /c306
- U3 pad 15: unconnected-(U3-C6-Pad15) -> /c307
- U3 pad 16: unconnected-(U3-C7-Pad16) -> /c308
- U3 pad 17: unconnected-(U3-C8-Pad17) -> /c309
- U3 pad 18: unconnected-(U3-C9-Pad18) -> /c310
- U3 pad 19: unconnected-(U3-C10-Pad19) -> /c311
- U3 pad 20: unconnected-(U3-C11-Pad20) -> /c312
- U3 pad 21: unconnected-(U3-C12-Pad21) -> /c313
- U3 pad 22: unconnected-(U3-C13-Pad22) -> /c314
- U3 pad 23: unconnected-(U3-C14-Pad23) -> /c315
- U3 pad 24: unconnected-(U3-C15-Pad24) -> /c316
- U3 pad 9: unconnected-(U3-C0-Pad9) -> /c301
- U4 pad 10: unconnected-(U4-C1-Pad10) -> /c402
- U4 pad 11: unconnected-(U4-C2-Pad11) -> /c403
- U4 pad 12: unconnected-(U4-C3-Pad12) -> /c404
- U4 pad 13: unconnected-(U4-C4-Pad13) -> /c405
- U4 pad 14: unconnected-(U4-C5-Pad14) -> /c406
- U4 pad 15: unconnected-(U4-C6-Pad15) -> /c407
- U4 pad 16: unconnected-(U4-C7-Pad16) -> /c408
- U4 pad 17: unconnected-(U4-C8-Pad17) -> /c409
- U4 pad 18: unconnected-(U4-C9-Pad18) -> /c410
- U4 pad 19: unconnected-(U4-C10-Pad19) -> /c411
- U4 pad 20: unconnected-(U4-C11-Pad20) -> /c412
- U4 pad 21: unconnected-(U4-C12-Pad21) -> /c413
- U4 pad 22: unconnected-(U4-C13-Pad22) -> /c414
- U4 pad 23: unconnected-(U4-C14-Pad23) -> /c415
- U4 pad 24: unconnected-(U4-C15-Pad24) -> /c416
- U4 pad 9: unconnected-(U4-C0-Pad9) -> /c401
Routing:
- net +3.3V: track 0.00 -> 156.1 mm
- net +5V: track 0.00 -> 146.6 mm
- net /S0: track 0.00 -> 117.5 mm, vias 0 -> 1
- net /S1: track 0.00 -> 115.3 mm, vias 0 -> 1
- net /S2: track 0.00 -> 112.9 mm, vias 0 -> 1
- net /S3: track 0.00 -> 109.7 mm, vias 0 -> 1
- net /SIG3: track 0.00 -> 56.4 mm
- net /c401: track 0.00 -> 56.3 mm
- net /c301: track 0.00 -> 56.3 mm
- net /c116: track 0.00 -> 55.4 mm
- net /c216: track 0.00 -> 55.3 mm
- net /c402: track 0.00 -> 50.3 mm
- net /c302: track 0.00 -> 50.3 mm
- net /c303: track 0.00 -> 50.2 mm
- net /c403: track 0.00 -> 50.2 mm
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- added copper zone on B.Cu, net GND
Other:
- board outline added: 128.8 x 57.2 mm
